File: noise-fob-no-fill.brd (EAGLE design)
At the start: 110.6 x 77 mm, 10 parts

Commit message: updates
Routing:
- net N$1: track 26.1 -> 27.2 mm
Changed lines of the file:
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@@
 <contactref element="U$2" pad="P$1"/>
 <contactref element="U$5" pad="P$1"/>
-<wire x1="31.242" y1="-58.42" x2="38.354" y2="-51.308" width="1.27" layer="16"/>
-<wire x1="19.05" y1="-67.818" x2="28.448" y2="-58.42" width="1.27" layer="16"/>
-<wire x1="28.448" y1="-58.42" x2="31.242" y2="-58.42" width="1.27" layer="16"/>
+<wire x1="38.1" y1="-53.34" x2="38.1" y2="-51.562" width="1.27" layer="16"/>
+<wire x1="38.1" y1="-51.562" x2="38.354" y2="-51.308" width="1.27" layer="16"/>
+<wire x1="35.56" y1="-53.34" x2="38.1" y2="-53.34" width="1.27" layer="16"/>
+<wire x1="19.05" y1="-67.818" x2="21.082" y2="-67.818" width="1.27" layer="16"/>
+<wire x1="21.082" y1="-67.818" x2="35.56" y2="-53.34" width="1.27" layer="16"/>
 </signal>
 <signal name="N$2">
@@
 <wire x1="53.34" y1="-55.88" x2="63.5" y2="-55.88" width="1.27" layer="16"/>
 <wire x1="45.72" y1="-53.34" x2="50.8" y2="-53.34" width="1.27" layer="16"/>
-<wire x1="26.67" y1="-65.786" x2="31.496" y2="-60.96" width="1.27" layer="16"/>
-<wire x1="31.496" y1="-60.96" x2="38.1" y2="-60.96" width="1.27" layer="16"/>
-<wire x1="38.1" y1="-60.96" x2="45.72" y2="-53.34" width="1.27" layer="16"/>
+<wire x1="26.67" y1="-65.786" x2="28.956" y2="-65.786" width="1.27" layer="16"/>
+<wire x1="33.528" y1="-61.214" x2="38.608" y2="-61.214" width="1.27" layer="16"/>
+<wire x1="38.608" y1="-61.214" x2="38.608" y2="-60.452" width="1.27" layer="16"/>
+<wire x1="38.608" y1="-60.452" x2="45.72" y2="-53.34" width="1.27" layer="16"/>
+<wire x1="28.956" y1="-65.786" x2="33.528" y2="-61.214" width="1.27" layer="16"/>
 </signal>
 <signal name="N$3">
@@
 <wire x1="66.04" y1="-29.21" x2="66.548" y2="-29.21" width="1.27" layer="16"/>
 </signal>
-<signal name="GND" airwireshidden="yes">
+<signal name="GND">
 <contactref element="U$2" pad="P$2"/>
 <contactref element="U$4" pad="P$2"/>
@@
 <contactref element="U$1" pad="P$2"/>
 <contactref element="U$8" pad="P$7"/>
-<polygon width="1.27" layer="16" isolate="0.889" thermals="no">
+<polygon width="1.27" layer="16" isolate="1.016">
 <vertex x="5.08" y="-88.9"/>
 <vertex x="121.92" y="-88.9"/>
